File: Electric/PCBs/fabFlipDriver/fabFlipDriver.kicad_sch (KiCad schematic)
At the start: 89 parts, among them J1 Conn_02x05_Odd_Even, J2 Conn_02x05_Odd_Even, J3 Conn_01x08, J4 Conn_01x08, J5 Conn_01x02, J6 Conn_01x02, J7 Conn_01x02, Q1 AO3401A, Q10 AO3401A, Q11 2N7002, Q12 2N7002, Q13 AO3401A, Q14 AO3401A, Q15 2N7002, Q16 2N7002, Q17 AO3401A, Q18 AO3401A, Q19 2N7002, Q2 AO3401A, Q20 2N7002, Q21 AO3401A, Q22 AO3401A, Q23 2N7002, Q24 2N7002, Q25 AO3401A, Q26 AO3401A, Q27 2N7002, Q28 2N7002, Q29 AO3401A, Q3 2N7002, Q30 AO3401A, Q31 2N7002, Q32 2N7002, Q4 2N7002, Q5 AO3401A, Q6 AO3401A, Q7 2N7002, Q8 2N7002, Q9 AO3401A, U1 74HC595, U2 74HC595

Commit message: PCB update
Connections:
- net Logic01 renamed Bit08
- net Logic02 renamed Bit09
- net Logic03 renamed Bit10
- net Logic04 renamed Bit11
- net Logic05 renamed Bit12
- net Logic06 renamed Bit13
- net Logic07 renamed Bit14
- net Logic08 renamed Bit15
- net Logic09 renamed Bit00
- net Logic10 renamed Bit01
- net Logic11 renamed Bit02
- net Logic12 renamed Bit03
- net Logic13 renamed Bit04
- net Logic14 renamed Bit05
- net Logic15 renamed Bit06
- net Logic16 renamed Bit07
- net Out01 renamed O_08
- net Out02 renamed O_09
- net Out03 renamed O_10
- net Out04 renamed O_11
- net Out05 renamed O_12
- net Out06 renamed O_13
- net Out07 renamed O_14
- net Out08 renamed O_15
- net Out09 renamed O_00
- net Out10 renamed O_01
- net Out11 renamed O_02
- net Out12 renamed O_03
- net Out13 renamed O_04
- net Out14 renamed O_05
- net Out15 renamed O_06
- net Out16 renamed O_07

Commit message: Small changes
Other:
- company: (none) -> Fablab Munich
- title: (none) -> fabFlipDriver
Changed lines of the file:
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@@
 (kicad_sch (version 20211123) (generator eeschema)
   (paper "A4")
+  (title_block
+    (title "fabFlipDriver")
+    (date "2023-01-26")
+    (rev "V001")
+    (company "Fablab Munich")
+    (comment 1 "@tinyledmatrix ")
+  )
   (junction (at 196.215 80.01) (diameter 0) (color 0 0 0 0)
   )
